Commit message: Updating xacro and favourites

File: description/picknik_ur.xacro (robot description, xacro)
@@ -7,4 +7,7 @@
   <material name="plastic">
     <color rgba="0.1 0.1 0.1 1" />
+  </material>
+  <material name="offwhite">
+    <color rgba="0.01 0.01 0.01 1" />
   </material>
   <link name="world" />
@@ -1167,55 +1170,13 @@
   <link name="table">
     <visual>
-      <origin rpy="0 0 0" xyz="0 0 0.025" />
-      <geometry>
-        <mesh
-          filename="package://picknik_accessories/descriptions/furniture/generic_table/wood_block.dae"
-          scale="0.125 0.125 0.00625"
-        />
-      </geometry>
-    </visual>
-    <visual>
-      <origin rpy="0 0 0" xyz="0.4 0.4 -0.2" />
-      <geometry>
-        <box size="0.04 0.04 0.45" />
-      </geometry>
-      <material name="grey">
-        <color rgba="0.1 0.1 0.1 1.0" />
-      </material>
-    </visual>
-    <visual>
-      <origin rpy="0 0 0" xyz="0.4 -0.4 -0.2" />
-      <geometry>
-        <box size="0.04 0.04 0.45" />
-      </geometry>
-      <material name="grey">
-        <color rgba="0.1 0.1 0.1 1.0" />
-      </material>
-    </visual>
-    <visual>
-      <origin rpy="0 0 0" xyz="-0.4 -0.4 -0.2" />
-      <geometry>
-        <box size="0.04 0.04 0.45" />
-      </geometry>
-      <material name="grey">
-        <color rgba="0.1 0.1 0.1 1.0" />
-      </material>
-    </visual>
-    <visual>
-      <origin rpy="0 0 0" xyz="-0.4 0.4 -0.2" />
-      <geometry>
-        <box size="0.04 0.04 0.45" />
-      </geometry>
-      <material name="grey">
-        <color rgba="0.1 0.1 0.1 1.0" />
-      </material>
-    </visual>
-    <collision>
-      <origin rpy="0 0 0" xyz="0 0 0" />
-      <geometry>
-        <mesh
-          filename="package://picknik_accessories/descriptions/furniture/generic_table/wood_block.dae"
-          scale="0.125 0.125 0.00625"
-        />
+      <origin rpy="0 0 0" xyz="0 0 -0.45" />
+      <geometry>
+        <box size="3.5 1 0.9" />
+      </geometry>
+    </visual>
+    <collision>
+      <origin rpy="0 0 0" xyz="0 0 -0.45" />
+      <geometry>
+        <box size="3.5 1 0.9" />
       </geometry>
     </collision>
